File: hardware/kicad/mainboard.kicad_sch (KiCad schematic)
At the start: 82 parts, among them J1 XT60PW, J10 Body NeoPixel, J11 Slip ring, J12 Charger XT30, J13 SPK L, J14 SPK R, J15 ESTOP, J16 I2C-A exp (ESP32), J17 I2C-B exp (RP2350), J2 DFR0601 ribbon 2x5, J3 DFR0601 ribbon 2x5, J4 Servo L, J5 Servo R, J6 IMU BMI160 SPI, J7 S2S AS5600/pot, J8 Dome encoder, J9 Hall, Q1 SQJ431EP P-FET RPP, U1 ESP-WROOM-32 DevKit 30p, U2 RP2350-Zero, U3 DFPlayer Mini, U5 AP7361C-33 3.3V LDO, U6 74AHCT125, U7 74LVC245A

Commit message: v10 KiCad mainboard: collision-aware placer, library footprints, ERC 0 errors, placed on the casing outline; boss coordinates for the casing model
Co-Authored-By: Claude Opus 5 (1M context) <noreply@anthropic.com>
Parts:
- added H5: M3 boss, MountingHole:MountingHole_3.2mm_M3_Pad, symbol ZCLASS:H5
Connections:
- net GND: now also H5.1

Commit message: v10 mainboard: true 2 mm outline offset (was 0.95 mm min), DFPlayer at tail tip with SD slot facing the opening, 6 V buck to left lobe, board title + credits on silkscreen, schematic title block; renders in docs
Co-Authored-By: Claude Opus 5 (1M context) <noreply@anthropic.com>
Other:
- company: Z-ClassControlSystem -> Z-Class Control System - James VanDusen
- title: Z-Class v10 mainboard -> Z-Drive v10.0 Mainboard
Changed lines of the file:
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@@
 (kicad_sch (version 20231120) (generator "zclass_gen") (generator_version "1.0")
   (paper "A2")
-  (title_block (title "Z-Class v10 mainboard") (company "Z-ClassControlSystem") (comment 1 "generated from hardware/netlist/mainboard.py"))
+  (title_block (title "Z-Drive v10.0 Mainboard") (company "Z-Class Control System - James VanDusen") (rev "A") (comment 1 "Special thanks to Mimir Reynisson, Greg Bellows and Joe Latiola") (comment 2 "Generated from hardware/netlist/mainboard.py - edit the netlist, not this file") (comment 3 "Modules: ESP-WROOM-32 DevKit, RP2350-Zero, DFPlayer Mini, Pololu D24V50F5 / D24V22F6, MAX9744 amp module"))
   (symbol (lib_id "ZCLASS:PS1") (at 72.39 48.26 0) (unit 1) (exclude_from_sim no) (in_bom yes) (on_board yes) (dnp no)
     (property "Reference" "PS1" (at 72.39 43.18 0) (effects (font (size 1.27 1.27))))

Commit message: v10 mainboard: DevKit right-column pinout corrected (3V3 at USB end), ESP32 antenna copper keep-out, 31 GND stitching vias, current-based netclasses (Power 3.0 mm, Audio 1.0, Motor 0.5), 10 A input fuse
Co-Authored-By: Claude Opus 5 (1M context) <noreply@anthropic.com>
Parts:
- F1: value 15A blade fuse -> 10A blade fuse
Connections:
- net DRIVE_INA: now also U1.25 (RX2); no longer U1.21 (RX2)
- net DRIVE_INB: now also U1.24 (TX2); no longer U1.22 (TX2)
- net DRIVE_PWM: now also U1.26 (D4); no longer U1.20 (D4)
- net GND: now also U1.29 (GND); no longer U1.17 (GND)
- net I2C_A_SCL: now also U1.28 (D15); no longer U1.18 (D15)
- net IMU_MISO: now also U1.21 (D19); no longer U1.25 (D19)
- net IMU_MOSI: now also U1.16 (D23); no longer U1.30 (D23)
- net IMU_SCK: now also U1.22 (D18); no longer U1.24 (D18)
- net LINK_ESP_TX: now also U1.20 (D21); no longer U1.26 (D21)
- net LINK_RP_TX: now also U1.17 (D22); no longer U1.29 (D22)
Changed lines of the file:
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@@
   (global_label "GND" (shape bidirectional) (at 59.69 115.57 180) (fields_autoplaced yes) (effects (font (size 1.27 1.27)) (justify right)) (property "Intersheetrefs" "${INTERSHEET_REFS}" (at 59.69 115.57 0) (effects (font (size 1.27 1.27)) (hide yes))))
   (global_label "+5V_LOGIC" (shape bidirectional) (at 59.69 118.11 180) (fields_autoplaced yes) (effects (font (size 1.27 1.27)) (justify right)) (property "Intersheetrefs" "${INTERSHEET_REFS}" (at 59.69 118.11 0) (effects (font (size 1.27 1.27)) (hide yes))))
-  (no_connect (at 85.09 82.55))
-  (global_label "GND" (shape bidirectional) (at 85.09 85.09 0) (fields_autoplaced yes) (effects (font (size 1.27 1.27)) (justify left)) (property "Intersheetrefs" "${INTERSHEET_REFS}" (at 85.09 85.09 0) (effects (font (size 1.27 1.27)) (hide yes))))
-  (global_label "I2C_A_SCL" (shape bidirectional) (at 85.09 87.63 0) (fields_autoplaced yes) (effects (font (size 1.27 1.27)) (justify left)) (property "Intersheetrefs" "${INTERSHEET_REFS}" (at 85.09 87.63 0) (effects (font (size 1.27 1.27)) (hide yes))))
+  (global_label "IMU_MOSI" (shape bidirectional) (at 85.09 82.55 0) (fields_autoplaced yes) (effects (font (size 1.27 1.27)) (justify left)) (property "Intersheetrefs" "${INTERSHEET_REFS}" (at 85.09 82.55 0) (effects (font (size 1.27 1.27)) (hide yes))))
+  (global_label "LINK_RP_TX" (shape bidirectional) (at 85.09 85.09 0) (fields_autoplaced yes) (effects (font (size 1.27 1.27)) (justify left)) (property "Intersheetrefs" "${INTERSHEET_REFS}" (at 85.09 85.09 0) (effects (font (size 1.27 1.27)) (hide yes))))
+  (no_connect (at 85.09 87.63))
   (no_connect (at 85.09 90.17))
-  (global_label "DRIVE_PWM" (shape bidirectional) (at 85.09 92.71 0) (fields_autoplaced yes) (effects (font (size 1.27 1.27)) (justify left)) (property "Intersheetrefs" "${INTERSHEET_REFS}" (at 85.09 92.71 0) (effects (font (size 1.27 1.27)) (hide yes))))
-  (global_label "DRIVE_INA" (shape bidirectional) (at 85.09 95.25 0) (fields_autoplaced yes) (effects (font (size 1.27 1.27)) (justify left)) (property "Intersheetrefs" "${INTERSHEET_REFS}" (at 85.09 95.25 0) (effects (font (size 1.27 1.27)) (hide yes))))
-  (global_label "DRIVE_INB" (shape bidirectional) (at 85.09 97.79 0) (fields_autoplaced yes) (effects (font (size 1.27 1.27)) (justify left)) (property "Intersheetrefs" "${INTERSHEET_REFS}" (at 85.09 97.79 0) (effects (font (size 1.27 1.27)) (hide yes))))
+  (global_label "LINK_ESP_TX" (shape bidirectional) (at 85.09 92.71 0) (fields_autoplaced yes) (effects (font (size 1.27 1.27)) (justify left)) (property "Intersheetrefs" "${INTERSHEET_REFS}" (at 85.09 92.71 0) (effects (font (size 1.27 1.27)) (hide yes))))
+  (global_label "IMU_MISO" (shape bidirectional) (at 85.09 95.25 0) (fields_autoplaced yes) (effects (font (size 1.27 1.27)) (justify left)) (property "Intersheetrefs" "${INTERSHEET_REFS}" (at 85.09 95.25 0) (effects (font (size 1.27 1.27)) (hide yes))))
+  (global_label "IMU_SCK" (shape bidirectional) (at 85.09 97.79 0) (fields_autoplaced yes) (effects (font (size 1.27 1.27)) (justify left)) (property "Intersheetrefs" "${INTERSHEET_REFS}" (at 85.09 97.79 0) (effects (font (size 1.27 1.27)) (hide yes))))
   (global_label "IMU_CS" (shape bidirectional) (at 85.09 100.33 0) (fields_autoplaced yes) (effects (font (size 1.27 1.27)) (justify left)) (property "Intersheetrefs" "${INTERSHEET_REFS}" (at 85.09 100.33 0) (effects (font (size 1.27 1.27)) (hide yes))))
-  (global_label "IMU_SCK" (shape bidirectional) (at 85.09 102.87 0) (fields_autoplaced yes) (effects (font (size 1.27 1.27)) (justify left)) (property "Intersheetrefs" "${INTERSHEET_REFS}" (at 85.09 102.87 0) (effects (font (size 1.27 1.27)) (hide yes))))
-  (global_label "IMU_MISO" (shape bidirectional) (at 85.09 105.41 0) (fields_autoplaced yes) (effects (font (size 1.27 1.27)) (justify left)) (property "Intersheetrefs" "${INTERSHEET_REFS}" (at 85.09 105.41 0) (effects (font (size 1.27 1.27)) (hide yes))))
-  (global_label "LINK_ESP_TX" (shape bidirectional) (at 85.09 107.95 0) (fields_autoplaced yes) (effects (font (size 1.27 1.27)) (justify left)) (property "Intersheetrefs" "${INTERSHEET_REFS}" (at 85.09 107.95 0) (effects (font (size 1.27 1.27)) (hide yes))))
+  (global_label "DRIVE_INB" (shape bidirectional) (at 85.09 102.87 0) (fields_autoplaced yes) (effects (font (size 1.27 1.27)) (justify left)) (property "Intersheetrefs" "${INTERSHEET_REFS}" (at 85.09 102.87 0) (effects (font (size 1.27 1.27)) (hide yes))))
+  (global_label "DRIVE_INA" (shape bidirectional) (at 85.09 105.41 0) (fields_autoplaced yes) (effects (font (size 1.27 1.27)) (justify left)) (property "Intersheetrefs" "${INTERSHEET_REFS}" (at 85.09 105.41 0) (effects (font (size 1.27 1.27)) (hide yes))))
+  (global_label "DRIVE_PWM" (shape bidirectional) (at 85.09 107.95 0) (fields_autoplaced yes) (effects (font (size 1.27 1.27)) (justify left)) (property "Intersheetrefs" "${INTERSHEET_REFS}" (at 85.09 107.95 0) (effects (font (size 1.27 1.27)) (hide yes))))
   (no_connect (at 85.09 110.49))
-  (no_connect (at 85.09 113.03))
-  (global_label "LINK_RP_TX" (shape bidirectional) (at 85.09 115.57 0) (fields_autoplaced yes) (effects (font (size 1.27 1.27)) (justify left)) (property "Intersheetrefs" "${INTERSHEET_REFS}" (at 85.09 115.57 0) (effects (font (size 1.27 1.27)) (hide yes))))
-  (global_label "IMU_MOSI" (shape bidirectional) (at 85.09 118.11 0) (fields_autoplaced yes) (effects (font (size 1.27 1.27)) (justify left)) (property "Intersheetrefs" "${INTERSHEET_REFS}" (at 85.09 118.11 0) (effects (font (size 1.27 1.27)) (hide yes))))
+  (global_label "I2C_A_SCL" (shape bidirectional) (at 85.09 113.03 0) (fields_autoplaced yes) (effects (font (size 1.27 1.27)) (justify left)) (property "Intersheetrefs" "${INTERSHEET_REFS}" (at 85.09 113.03 0) (effects (font (size 1.27 1.27)) (hide yes))))
+  (global_label "GND" (shape bidirectional) (at 85.09 115.57 0) (fields_autoplaced yes) (effects (font (size 1.27 1.27)) (justify left)) (property "Intersheetrefs" "${INTERSHEET_REFS}" (at 85.09 115.57 0) (effects (font (size 1.27 1.27)) (hide yes))))
+  (no_connect (at 85.09 118.11))
   (symbol (lib_id "ZCLASS:U2") (at 72.39 147.32 0) (unit 1) (exclude_from_sim no) (in_bom yes) (on_board yes) (dnp no)
     (property "Reference" "U2" (at 72.39 129.54 0) (effects (font (size 1.27 1.27))))
@@
   (symbol (lib_id "ZCLASS:F1") (at 143.51 181.61 0) (unit 1) (exclude_from_sim no) (in_bom yes) (on_board yes) (dnp no)
     (property "Reference" "F1" (at 143.51 177.80 0) (effects (font (size 1.27 1.27))))
-    (property "Value" "15A blade fuse" (at 143.51 185.42 0) (effects (font (size 1.27 1.27))))
+    (property "Value" "10A blade fuse" (at 143.51 185.42 0) (effects (font (size 1.27 1.27))))
     (property "Footprint" "ZCLASS:Fuse_Mini_Blade" (at 143.51 181.61 0) (effects (font (size 1.27 1.27)) (hide yes)))
     (property "Datasheet" "" (at 143.51 181.61 0) (effects (font (size 1.27 1.27)) (hide yes)))

Commit message: v10 mainboard: 4-layer routed ~95% (F/B GND pours + In1 GND/In2 +5V planes), 7.4V servo rail (D24V25F7); 27 signal/plane opens + 11 edge tracks remain for interactive GUI finish
Co-Authored-By: Claude Opus 5 (1M context) <noreply@anthropic.com>
Parts:
- C4: value 470u/10V -> 470u/16V
- PS2: value Pololu D24V22F6 6V 2.5A -> Pololu D24V25F7 7.5V 2.5A
Connections:
- net +6V_SERVO renamed +7V4_SERVO
Changed lines of the file:
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@@
   (symbol (lib_id "ZCLASS:PS2") (at 72.39 66.04 0) (unit 1) (exclude_from_sim no) (in_bom yes) (on_board yes) (dnp no)
     (property "Reference" "PS2" (at 72.39 60.96 0) (effects (font (size 1.27 1.27))))
-    (property "Value" "Pololu D24V22F6 6V 2.5A" (at 72.39 71.12 0) (effects (font (size 1.27 1.27))))
+    (property "Value" "Pololu D24V25F7 7.5V 2.5A" (at 72.39 71.12 0) (effects (font (size 1.27 1.27))))
     (property "Footprint" "ZCLASS:Pololu_D24V22F6" (at 72.39 66.04 0) (effects (font (size 1.27 1.27)) (hide yes)))
     (property "Datasheet" "" (at 72.39 66.04 0) (effects (font (size 1.27 1.27)) (hide yes)))
@@
   (global_label "VIN" (shape bidirectional) (at 59.69 64.77 180) (fields_autoplaced yes) (effects (font (size 1.27 1.27)) (justify right)) (property "Intersheetrefs" "${INTERSHEET_REFS}" (at 59.69 64.77 0) (effects (font (size 1.27 1.27)) (hide yes))))
   (global_label "GND" (shape bidirectional) (at 59.69 67.31 180) (fields_autoplaced yes) (effects (font (size 1.27 1.27)) (justify right)) (property "Intersheetrefs" "${INTERSHEET_REFS}" (at 59.69 67.31 0) (effects (font (size 1.27 1.27)) (hide yes))))
-  (global_label "+6V_SERVO" (shape bidirectional) (at 85.09 64.77 0) (fields_autoplaced yes) (effects (font (size 1.27 1.27)) (justify left)) (property "Intersheetrefs" "${INTERSHEET_REFS}" (at 85.09 64.77 0) (effects (font (size 1.27 1.27)) (hide yes))))
+  (global_label "+7V4_SERVO" (shape bidirectional) (at 85.09 64.77 0) (fields_autoplaced yes) (effects (font (size 1.27 1.27)) (justify left)) (property "Intersheetrefs" "${INTERSHEET_REFS}" (at 85.09 64.77 0) (effects (font (size 1.27 1.27)) (hide yes))))
   (no_connect (at 85.09 67.31))
   (symbol (lib_id "ZCLASS:U1") (at 72.39 100.33 0) (unit 1) (exclude_from_sim no) (in_bom yes) (on_board yes) (dnp no)
@@
   )
   (global_label "SERVO_L" (shape bidirectional) (at 59.69 511.81 180) (fields_autoplaced yes) (effects (font (size 1.27 1.27)) (justify right)) (property "Intersheetrefs" "${INTERSHEET_REFS}" (at 59.69 511.81 0) (effects (font (size 1.27 1.27)) (hide yes))))
-  (global_label "+6V_SERVO" (shape bidirectional) (at 59.69 514.35 180) (fields_autoplaced yes) (effects (font (size 1.27 1.27)) (justify right)) (property "Intersheetrefs" "${INTERSHEET_REFS}" (at 59.69 514.35 0) (effects (font (size 1.27 1.27)) (hide yes))))
+  (global_label "+7V4_SERVO" (shape bidirectional) (at 59.69 514.35 180) (fields_autoplaced yes) (effects (font (size 1.27 1.27)) (justify right)) (property "Intersheetrefs" "${INTERSHEET_REFS}" (at 59.69 514.35 0) (effects (font (size 1.27 1.27)) (hide yes))))
   (global_label "GND" (shape bidirectional) (at 85.09 511.81 0) (fields_autoplaced yes) (effects (font (size 1.27 1.27)) (justify left)) (property "Intersheetrefs" "${INTERSHEET_REFS}" (at 85.09 511.81 0) (effects (font (size 1.27 1.27)) (hide yes))))
   (symbol (lib_id "ZCLASS:J5") (at 72.39 530.86 0) (unit 1) (exclude_from_sim no) (in_bom yes) (on_board yes) (dnp no)
@@
   )
   (global_label "SERVO_R" (shape bidirectional) (at 59.69 529.59 180) (fields_autoplaced yes) (effects (font (size 1.27 1.27)) (justify right)) (property "Intersheetrefs" "${INTERSHEET_REFS}" (at 59.69 529.59 0) (effects (font (size 1.27 1.27)) (hide yes))))
-  (global_label "+6V_SERVO" (shape bidirectional) (at 59.69 532.13 180) (fields_autoplaced yes) (effects (font (size 1.27 1.27)) (justify right)) (property "Intersheetrefs" "${INTERSHEET_REFS}" (at 59.69 532.13 0) (effects (font (size 1.27 1.27)) (hide yes))))
+  (global_label "+7V4_SERVO" (shape bidirectional) (at 59.69 532.13 180) (fields_autoplaced yes) (effects (font (size 1.27 1.27)) (justify right)) (property "Intersheetrefs" "${INTERSHEET_REFS}" (at 59.69 532.13 0) (effects (font (size 1.27 1.27)) (hide yes))))
   (global_label "GND" (shape bidirectional) (at 85.09 529.59 0) (fields_autoplaced yes) (effects (font (size 1.27 1.27)) (justify left)) (property "Intersheetrefs" "${INTERSHEET_REFS}" (at 85.09 529.59 0) (effects (font (size 1.27 1.27)) (hide yes))))
   (symbol (lib_id "ZCLASS:J6") (at 143.51 49.53 0) (unit 1) (exclude_from_sim no) (in_bom yes) (on_board yes) (dnp no)
@@
   (symbol (lib_id "ZCLASS:C4") (at 143.51 379.73 0) (unit 1) (exclude_from_sim no) (in_bom yes) (on_board yes) (dnp no)
     (property "Reference" "C4" (at 143.51 375.92 0) (effects (font (size 1.27 1.27))))
-    (property "Value" "470u/10V" (at 143.51 383.54 0) (effects (font (size 1.27 1.27))))
+    (property "Value" "470u/16V" (at 143.51 383.54 0) (effects (font (size 1.27 1.27))))
     (property "Footprint" "Capacitor_SMD:CP_Elec_8x10" (at 143.51 379.73 0) (effects (font (size 1.27 1.27)) (hide yes)))
     (property "Datasheet" "" (at 143.51 379.73 0) (effects (font (size 1.27 1.27)) (hide yes)))
@@
     (instances (project "mainboard" (path "/0b82c761-6368-5a59-877e-dce7a78c7d89" (reference "C4") (unit 1))))
   )
-  (global_label "+6V_SERVO" (shape bidirectional) (at 130.81 379.73 180) (fields_autoplaced yes) (effects (font (size 1.27 1.27)) (justify right)) (property "Intersheetrefs" "${INTERSHEET_REFS}" (at 130.81 379.73 0) (effects (font (size 1.27 1.27)) (hide yes))))
+  (global_label "+7V4_SERVO" (shape bidirectional) (at 130.81 379.73 180) (fields_autoplaced yes) (effects (font (size 1.27 1.27)) (justify right)) (property "Intersheetrefs" "${INTERSHEET_REFS}" (at 130.81 379.73 0) (effects (font (size 1.27 1.27)) (hide yes))))
   (global_label "GND" (shape bidirectional) (at 156.21 379.73 0) (fields_autoplaced yes) (effects (font (size 1.27 1.27)) (justify left)) (property "Intersheetrefs" "${INTERSHEET_REFS}" (at 156.21 379.73 0) (effects (font (size 1.27 1.27)) (hide yes))))
   (symbol (lib_id "ZCLASS:C5") (at 143.51 394.97 0) (unit 1) (exclude_from_sim no) (in_bom yes) (on_board yes) (dnp no)
