File: hardware/kicad/compact/mainboard.kicad_pcb (KiCad board)
At the start: 4 copper layers, 151.8 x 109.6 mm, 83 parts, among them J1 XT60PB-M vertical, J10 Body NeoPixel, J11 Slip ring (body lights), J13 SPK L, J14 SPK R, J15 ESTOP, J17 I2C-B exp (RP2350), J2 DFR0601 ribbon 2x5, J3 DFR0601 ribbon 2x5, J4 Servo L, J5 Servo R, J6 IMU BMI160 I2C, J7 S2S AS5600/pot, J8 Dome encoder, J9 Hall, Q1 Si7461DP P-FET RPP, U3 DFPlayer Mini, U5 AP7361C-33 3.3V LDO, U6 74AHCT125, U7 74LVC245A

Commit message: v10 mainboard r7: fix U7 74LVC245 direction (DIR -> +3V3, A->B), tie unused A3..A8 to GND
DIR was strapped to GND, which per the SN74LVC245A pin table is B->A: the 5 V dome
encoder on A1/A2 would never reach the RP2350 on B1/B2 and U7's A outputs would fight
the encoder. Pad 1 is now +3V3 via a 0.2 mm jumper around the package end to pin 20;
A3..A8 (inputs once DIR=H) run along the row to pin 10 GND. Compact board still
0 DRC errors (17 warnings, 2 cosmetic zone-island lines). Extended board synced.
Regenerated both schematics (compact's was stale) and the JLCPCB package
(ZDrive_v10_compact_*_r7.zip; BOM/CPL unchanged from the r6 upload).

Rev-A boards built from r6 gerbers: cut the GND spoke into U7 pin 1 and bridge pin 1
to pin 20.

Co-Authored-By: Claude Fable 5 <noreply@anthropic.com>
Connections:
- U7 pad 1: GND -> +3V3
- U7 pad 4: (no net) -> GND
- U7 pad 5: (no net) -> GND
- U7 pad 6: (no net) -> GND
- U7 pad 7: (no net) -> GND
- U7 pad 8: (no net) -> GND
- U7 pad 9: (no net) -> GND
Routing:
- net +3V3: track 419.5 -> 427.1 mm
- net GND: track 7.51 -> 11.4 mm
Changed lines of the file:
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@@
 			(layers "F.Cu" "F.Mask" "F.Paste")
 			(roundrect_rratio 0.25)
-			(net "GND")
+			(net "+3V3")
 		)
 		(pad "2" smd roundrect
@@
 			(layers "F.Cu" "F.Mask" "F.Paste")
 			(roundrect_rratio 0.25)
+			(net "GND")
 		)
 		(pad "5" smd roundrect
@@
 			(layers "F.Cu" "F.Mask" "F.Paste")
 			(roundrect_rratio 0.25)
+			(net "GND")
 		)
 		(pad "6" smd roundrect
@@
 			(layers "F.Cu" "F.Mask" "F.Paste")
 			(roundrect_rratio 0.25)
+			(net "GND")
 		)
 		(pad "7" smd roundrect
@@
 			(layers "F.Cu" "F.Mask" "F.Paste")
 			(roundrect_rratio 0.25)
+			(net "GND")
 		)
 		(pad "8" smd roundrect
@@
 			(layers "F.Cu" "F.Mask" "F.Paste")
 			(roundrect_rratio 0.25)
+			(net "GND")
 		)
 		(pad "9" smd roundrect
@@
 			(layers "F.Cu" "F.Mask" "F.Paste")
 			(roundrect_rratio 0.25)
+			(net "GND")
 		)
 		(pad "10" smd roundrect
@@
 	)
 	(segment
+		(start 209.25 155.35)
+		(end 209.25 159.25)
+		(width 0.2)
+		(layer "F.Cu")
+		(net "GND")
+	)
+	(segment
 		(start 209.05 125.541)
 		(end 210.678 127.169)
@@
 	)
 	(segment
+		(start 209.25 152.5)
+		(end 214.975 152.5)
+		(width 0.2)
+		(layer "F.Cu")
+		(net "+3V3")
+	)
+	(segment
 		(start 219.186 135.961)
 		(end 222.475 139.25)
@@
 		(layer "F.Cu")
 		(net "+3V3")
+	)
+	(segment
+		(start 214.975 152.5)
+		(end 214.975 153.4)
+		(width 0.2)
+		(layer "F.Cu")
+		(net "+3V3")
+	)
+	(segment
+		(start 209.25 153.4)
+		(end 209.25 152.5)
+		(width 0.2)
+		(layer "F.Cu")
+		(net "+3V3")
