File: hardware/kicad/compact/mainboard.kicad_sch (KiCad schematic)
At the start: 83 parts, among them J1 XT60PW, J10 Body NeoPixel, J11 Slip ring, J12 Charger XT30, J13 SPK L, J14 SPK R, J15 ESTOP, J16 I2C-A exp (ESP32), J17 I2C-B exp (RP2350), J2 DFR0601 ribbon 2x5, J3 DFR0601 ribbon 2x5, J4 Servo L, J5 Servo R, J6 IMU BMI160 SPI, J7 S2S AS5600/pot, J8 Dome encoder, J9 Hall, Q1 SQJ431EP P-FET RPP, U1 ESP-WROOM-32 DevKit 30p, U2 RP2350-Zero, U3 DFPlayer Mini, U5 AP7361C-33 3.3V LDO, U6 74AHCT125, U7 74LVC245A

Commit message: v10 mainboard: compact board routed, DRC-clean and packaged for JLCPCB (r6); extended variant split out
Two variants from one netlist (hardware/netlist/mainboard.py):
- hardware/kicad/compact/  original-casing outline (152x110). Hand-placed by James, autorouted
  (prep_route -> Freerouting 2.3 -> post_route), last nets finished in pcbnew. KiCad 10 DRC: 0 errors.
- hardware/kicad/extended/ casing +15 mm down (152x125), auto-placed, unrouted.

Design changes since 850cb81 (all verified against datasheets / vendor drawings):
- Input: single 12 V XT60 (now VERTICAL XT60PB-M, KiCad AMASS footprint) -> F1 10 A -> Q1 Si7461DP
  high-side RPP with the REAL PowerPAK pinout (1-3 S, 4 G, 5 D; the old mapping shorted BAT+ to GND)
  + D6 12 V gate zener / R33. D2 SS14 orientation fixed. BAT54S clamp + 100n on VBAT_SENSE.
- Charge path REMOVED (pack charges via its own lead): J12, F2, CHG nets, R26/R27 gone; slip ring
  J11 = XH 2-pin +5V_LED/GND. J16 removed (I2C-A on J7 pins 4/5).
- Servo rail 6.0 V (PS2 D24V25F6) for Hitec HS-805BB / JX HV2060MG. Pololu footprints = real 5-pin
  EN VIN GND GND OUT row. U5 = AMS1117-3.3 (pinout as routed; AP7361C-33E-13 is IN/GND/OUT - wrong).
- IMU J6 = XH 4-pin I2C (5V GND SCL SDA, v9.15 MPU order) for a GY-BMI160; ESP32 SPI pins freed.
- J8 dome encoder keeps the v9.15 order (B A GND 5V). J2/J3 bare 2x5 headers, J_AMP 2x7 with Vi2c.
- Modules socketed: U1 -> J_U1A/J_U1B (1x15), U2 -> J_U2A/J_U2B/J_U2C (1x9,1x9,1x5), pads
  coincident with the old module pads. L1 -> BLM31KN601SN1L (2.9 A). F1 = Keystone 3568 holder.
- Netclasses: Default 0.15/0.25, Rail 0.6 (+5V_LOGIC,+3V3); In2 = signal layer with +5V pour
  (routed as a net). Antenna keep-out trimmed so H3 clears it. Axle keep-out disc for routing.

Fab package hardware/fab/compact-20260823 + ZDrive_v10_compact_{GERBERS,JLCPCB}_r6.zip:
Gerbers (page origin, no drill map - JLC's previewer needs both), JLC-format BOM (38/38 lines with
verified LCSC numbers) and CPL (centroids, +90 deg for Pin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
Parts:
- removed F2: 3A fuse, Fuse:Fuse_1206_3216Metric, symbol ZCLASS:F2
- removed J12: Charger XT30, ZCLASS:XT30PW, symbol ZCLASS:J12
- removed J16: I2C-A exp (ESP32), Connector_JST:JST_SH_SM04B-SRSS-TB_1x04-1MP_P1.00mm_Horizontal, symbol ZCLASS:J16
- removed R26: 47k, Resistor_SMD:R_0603_1608Metric, symbol ZCLASS:R26
- removed R27: 10k, Resistor_SMD:R_0603_1608Metric, symbol ZCLASS:R27
- added C29: 100n, Capacitor_SMD:C_0603_1608Metric, symbol ZCLASS:C29
- added D4: BAT54S, Package_TO_SOT_SMD:SOT-23, symbol ZCLASS:D4
- added D6: BZT52C12 12V zener, Diode_SMD:D_SOD-123, symbol ZCLASS:D6
- added R33: 47k, Resistor_SMD:R_0603_1608Metric, symbol ZCLASS:R33
- J11: value Slip ring -> Slip ring (body lights); footprint Connector_JST:JST_VH_B4P-VH_1x04_P3.96mm_Vertical -> Connector_JST:JST_VH_B2P-VH_1x02_P3.96mm_Vertical
- J4, J5: footprint Connector_JST:JST_XH_B3B-XH-A_1x03_P2.50mm_Vertical -> Connector_PinHeader_2.54mm:PinHeader_1x03_P2.54mm_Vertical
- Q1: value SQJ431EP P-FET RPP -> Si7461DP P-FET RPP
Connections:
- net +3V3: now also D4.2 (K2)
- net +5V_LOGIC: now also D2.2, J8.4 (5V); no longer D2.1, J8.1 (5V)
- net BAT_F: now also Q1.5 (D); no longer Q1.1 (S)
- net ENC_A_5V: now also J8.2 (A); no longer J8.3 (A)
- net ENC_B_5V: now also J8.1 (B); no longer J8.4 (B)
- net GND: now also J8.3 (GND), C29.2, D4.1 (A1), R33.2; no longer J8.2 (GND), Q1.3 (G)
- net RP_5V: now also D2.1; no longer D2.2
- net VBAT_SENSE: now also C29.1, D4.3 (COM)
- net VIN: now also Q1.1 (S), Q1.3 (S), D6.1
- removed net CHG+: J11.3 (CHG+)
- removed net CHG-: J11.4 (CHG-)
- net CHG_SENSE: no longer names the net of U1.3 (VN)
- new net Q1_G: D6.2, Q1.4 (G), R33.1
- no-connect marks 34 -> 35
Other:
- moved on the sheet: C1, C10, C11, C12, C2, C26, C27, C28, C3, C4, C5, C6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

Commit message: v10 mainboard r7: fix U7 74LVC245 direction (DIR -> +3V3, A->B), tie unused A3..A8 to GND
DIR was strapped to GND, which per the SN74LVC245A pin table is B->A: the 5 V dome
encoder on A1/A2 would never reach the RP2350 on B1/B2 and U7's A outputs would fight
the encoder. Pad 1 is now +3V3 via a 0.2 mm jumper around the package end to pin 20;
A3..A8 (inputs once DIR=H) run along the row to pin 10 GND. Compact board still
0 DRC errors (17 warnings, 2 cosmetic zone-island lines). Extended board synced.
Regenerated both schematics (compact's was stale) and the JLCPCB package
(ZDrive_v10_compact_*_r7.zip; BOM/CPL unchanged from the r6 upload).

Rev-A boards built from r6 gerbers: cut the GND spoke into U7 pin 1 and bridge pin 1
to pin 20.

Co-Authored-By: Claude Fable 5 <noreply@anthropic.com>
Parts:
- removed R31: 33R, Resistor_SMD:R_0603_1608Metric, symbol ZCLASS:R31
- removed R32: 33R, Resistor_SMD:R_0603_1608Metric, symbol ZCLASS:R32
- removed U1: ESP-WROOM-32 DevKit 30p, ZCLASS:DevKit_2x15_25.4mm, symbol ZCLASS:U1
- removed U2: RP2350-Zero, ZCLASS:RP2350_Zero, symbol ZCLASS:U2
- added J_U1A: ESP32 DevKitC socket L (1x15), Connector_PinSocket_2.54mm:PinSocket_1x15_P2.54mm_Vertical, symbol ZCLASS:J_U1A
- added J_U1B: ESP32 DevKitC socket R (1x15), Connector_PinSocket_2.54mm:PinSocket_1x15_P2.54mm_Vertical, symbol ZCLASS:J_U1B
- added J_U2A: RP2350-Zero socket L (1x9), Connector_PinSocket_2.54mm:PinSocket_1x09_P2.54mm_Vertical, symbol ZCLASS:J_U2A
- added J_U2B: RP2350-Zero socket R (1x9), Connector_PinSocket_2.54mm:PinSocket_1x09_P2.54mm_Vertical, symbol ZCLASS:J_U2B
- added J_U2C: RP2350-Zero socket end (1x5), Connector_PinSocket_2.54mm:PinSocket_1x05_P2.54mm_Vertical, symbol ZCLASS:J_U2C
- J1: value XT60PW -> XT60PB-M vertical; footprint ZCLASS:XT60PW -> Connector_AMASS:AMASS_XT60-M_1x02_P7.20mm_Vertical
- J11: footprint Connector_JST:JST_VH_B2P-VH_1x02_P3.96mm_Vertical -> Connector_JST:JST_XH_B2B-XH-A_1x02_P2.50mm_Vertical
- J2, J3: footprint ZCLASS:Hdr_2x5_shrouded -> Connector_PinHeader_2.54mm:PinHeader_2x05_P2.54mm_Vertical
- J6: value IMU BMI160 SPI -> IMU BMI160 I2C; footprint Connector_JST:JST_SH_SM06B-SRSS-TB_1x06-1MP_P1.00mm_Horizontal -> Connector_JST:JST_XH_B4B-XH-A_1x04_P2.50mm_Vertical
- J_AMP: footprint ZCLASS:Hdr_2x6 -> Connector_PinHeader_2.54mm:PinHeader_2x07_P2.54mm_Vertical
- PS2: value Pololu D24V25F7 7.5V 2.5A -> Pololu D24V25F6 6V 2.5A; footprint ZCLASS:Pololu_D24V22F6 -> ZCLASS:Pololu_D24V25F6
Connections:
- net IMU_MISO is gone; now on net I2C_A_SDA: J6.4 (SDA)
- net IMU_SCK_R is gone; now on net I2C_A_SCL: J6.3 (SCL)
- net +3V3: now also J_AMP.13 (VI2C), U7.1 (DIR); no longer J6.1 (3V3)
- net +5V_LOGIC: now also J6.1 (5V), PS1.5 (VOUT), J_U1A.15 (VIN); no longer PS1.3 (VOUT)
- net AMP_SHDN: now also J_U2B.3 (GP2)
- net DF_BUSY: now also J_U2A.8 (GP15)
- net DF_RX_RP: now also J_U2B.6 (GP5)
- net DF_TX_RP: now also J_U2B.5 (GP4)
- net DOME_INA: now also J_U2C.1 (GP9)
- net DOME_INB: now also J_U2C.2 (GP10)
- net DOME_PWM: now also J_U2B.9 (GP8)
- net DRIVE_INA: now also J_U1B.10 (RX2)
- net DRIVE_INB: now also J_U1B.9 (TX2)
- net DRIVE_PWM: now also J_U1B.11 (D4)
- net ENC_A_3V3: now also J_U2C.3 (GP11)
- net ENC_B_3V3: now also J_U2C.4 (GP12)
- net ESTOP_SENSE: now also J_U1A.2 (VP)
- net FLY_INA: now also J_U1A.7 (D33)
- net FLY_INB: now also J_U1A.11 (D14)
- net FLY_PWM: now also J_U1A.6 (D32)
- net GND: now also J_AMP.14 (GND), PS1.3 (GND), PS1.4 (GND), PS2.3 (GND), PS2.4 (GND), U7.4 (A3), U7.5 (A4), U7.6 (A5), U7.7 (A6), U7.8 (A7), U7.9 (A8), J_U1A.14 (GND), J_U1B.14 (GND), J_U2A.2 (GND); no longer PS1.2 (GND), PS2.2 (GND), U7.1 (DIR)
- net HALL: now also J_U2C.5 (GP13)
- net I2C_A_SCL: now also J_U1B.13 (D15)
- net I2C_A_SDA: now also J_U1A.13 (D13)
- net I2C_B_SCL: now also J_U2A.6 (GP27)
- net I2C_B_SDA: now also J_U2A.7 (GP26)
- net LINK_ESP_TX: now also J_U1B.5 (D21), J_U2B.2 (GP1)
- net LINK_RP_TX: now also J_U1B.2 (D22), J_U2B.1 (GP0)
- net NEO_3V3: now also J_U2A.9 (GP14)
- net RP_5V: now also J_U2A.1 (5V)
- net S2S_INA: now also J_U1A.9 (D26)
- net S2S_INB: now also J_U1A.10 (D27)
- net S2S_POS: now also J_U1A.4 (D34)
- net S2S_PWM: now also J_U1A.8 (D25)
- net SERVO_L: now also J_U2B.7 (GP6)
- net SERVO_R: now also J_U2B.8 (GP7)
- net V5_SENSE: now also J_U2A.5 (GP28)
- net VBAT_SENSE: now also J_U1A.5 (D35)
- net VIN: now also PS1.2 (VIN), PS2.2 (VIN); no longer PS1.1 (VIN), PS2.1 (VIN)
- net +7V4_SERVO renamed +6V_SERVO
- net +6V_SERVO: now also PS2.5 (VOUT); no longer PS2.3 (VOUT)
- removed net IMU_CS: J6.6 (CS)
- removed net IMU_MOSI_R: J6.5 (MOSI)
- no-connect marks 35 -> 33
Other:
- moved on the sheet: C1, C10, C11, C12, C2, C26, C27, C28, C29, C3, C4, C5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
