File: hardware/kicad/extended/mainboard.kicad_pcb (KiCad board)
At the start: 4 copper layers, 151.8 x 124.6 mm, 83 parts, among them J1 XT60PB-M vertical, J10 Body NeoPixel, J11 Slip ring (body lights), J13 SPK L, J14 SPK R, J15 ESTOP, J17 I2C-B exp (RP2350), J2 DFR0601 ribbon 2x5, J3 DFR0601 ribbon 2x5, J4 Servo L, J5 Servo R, J6 IMU BMI160 I2C, J7 S2S AS5600/pot, J8 Dome encoder, J9 Hall, Q1 Si7461DP P-FET RPP, U3 DFPlayer Mini, U5 AP7361C-33 3.3V LDO, U6 74AHCT125, U7 74LVC245A

Commit message: v10 mainboard r7: fix U7 74LVC245 direction (DIR -> +3V3, A->B), tie unused A3..A8 to GND
DIR was strapped to GND, which per the SN74LVC245A pin table is B->A: the 5 V dome
encoder on A1/A2 would never reach the RP2350 on B1/B2 and U7's A outputs would fight
the encoder. Pad 1 is now +3V3 via a 0.2 mm jumper around the package end to pin 20;
A3..A8 (inputs once DIR=H) run along the row to pin 10 GND. Compact board still
0 DRC errors (17 warnings, 2 cosmetic zone-island lines). Extended board synced.
Regenerated both schematics (compact's was stale) and the JLCPCB package
(ZDrive_v10_compact_*_r7.zip; BOM/CPL unchanged from the r6 upload).

Rev-A boards built from r6 gerbers: cut the GND spoke into U7 pin 1 and bridge pin 1
to pin 20.

Co-Authored-By: Claude Fable 5 <noreply@anthropic.com>
Connections:
- U7 pad 1: GND -> +3V3
- U7 pad 4: (no net) -> GND
- U7 pad 5: (no net) -> GND
- U7 pad 6: (no net) -> GND
- U7 pad 7: (no net) -> GND
- U7 pad 8: (no net) -> GND
- U7 pad 9: (no net) -> GND
